File: kicad/timer.sch (KiCad schematic (older format))
At the start: 33 parts, among them IC1 STM8S003F3P, J1 PISK, J2 USB_OTG, J3 CONN_01X02, P1 kn1, P2 bat, P3 kn1, Q1 BC807-40, Q2 BC807-40, Q3 BC807-40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

Commit message: start
Parts:
- removed Q1, Q2, Q3: BC807-40, TO_SOT_Packages_SMD:SOT-23, symbol BC807-40
- removed R1, R3, R7: 4k7, Resistors_SMD:R_0603_HandSoldering, symbol R_Small
Connections:
- net c1: now also AFF1.12 (CA1)
- net c2: now also AFF1.9 (CA2)
- net c3: now also AFF1.8 (CA3)
Changed lines of the file:
@@
 LIBS:stm8
 LIBS:mylibkicad
-LIBS:kubik-cache
+LIBS:timer-cache
 EELAYER 25 0
 EELAYER END
@@
 Text Label 5600 2900 0    60   ~ 0
 dp
-$Comp
-L BC807-40 Q1
-U 1 1 58C44DC0
-P 7300 3250
-F 0 "Q1" H 7500 3325 50  0000 L CNN
-F 1 "BC807-40" H 7500 3250 50  0000 L CNN
-F 2 "TO_SOT_Packages_SMD:SOT-23" H 7500 3175 50  0000 L CIN
-F 3 "" H 7300 3250 50  0000 L CNN
-	1    7300 3250
-	1    0    0    1
-$EndComp
-$Comp
-L BC807-40 Q2
-U 1 1 58C45032
-P 7800 3250
-F 0 "Q2" H 8000 3325 50  0000 L CNN
-F 1 "BC807-40" H 8000 3250 50  0000 L CNN
-F 2 "TO_SOT_Packages_SMD:SOT-23" H 8000 3175 50  0000 L CIN
-F 3 "" H 7800 3250 50  0000 L CNN
-	1    7800 3250
-	1    0    0    1
-$EndComp
-$Comp
-L BC807-40 Q3
-U 1 1 58C450A4
-P 8300 3250
-F 0 "Q3" H 8500 3325 50  0000 L CNN
-F 1 "BC807-40" H 8500 3250 50  0000 L CNN
-F 2 "TO_SOT_Packages_SMD:SOT-23" H 8500 3175 50  0000 L CIN
-F 3 "" H 8300 3250 50  0000 L CNN
-	1    8300 3250
-	1    0    0    1
-$EndComp
-$Comp
-L VDD #PWR05
-U 1 1 58C454A6
-P 9000 2900
-F 0 "#PWR05" H 9000 2750 50  0001 C CNN
-F 1 "VDD" H 9000 3050 50  0000 C CNN
-F 2 "" H 9000 2900 50  0000 C CNN
-F 3 "" H 9000 2900 50  0000 C CNN
-	1    9000 2900
-	0    1    1    0
-$EndComp
-$Comp
-L R_Small R1
-U 1 1 58C4579E
-P 7100 3050
-F 0 "R1" H 7130 3070 50  0000 L CNN
-F 1 "4k7" H 7130 3010 50  0000 L CNN
-F 2 "Resistors_SMD:R_0603_HandSoldering" H 7100 3050 50  0000 C CNN
-F 3 "" H 7100 3050 50  0000 C CNN
-	1    7100 3050
-	1    0    0    -1
-$EndComp
-$Comp
-L R_Small R3
-U 1 1 58C4589D
-P 7600 3050
-F 0 "R3" H 7630 3070 50  0000 L CNN
-F 1 "4k7" H 7630 3010 50  0000 L CNN
-F 2 "Resistors_SMD:R_0603_HandSoldering" H 7600 3050 50  0000 C CNN
-F 3 "" H 7600 3050 50  0000 C CNN
-	1    7600 3050
-	1    0    0    -1
-$EndComp
-$Comp
-L R_Small R7
-U 1 1 58C45A71
-P 8100 3050
-F 0 "R7" H 8130 3070 50  0000 L CNN
-F 1 "4k7" H 8130 3010 50  0000 L CNN
-F 2 "Resistors_SMD:R_0603_HandSoldering" H 8100 3050 50  0000 C CNN
-F 3 "" H 8100 3050 50  0000 C CNN
-	1    8100 3050
-	1    0    0    -1
-$EndComp
 Text Label 7100 2650 0    60   ~ 0
 c1
@@
 	7400 3450 7400 3600
 Wire Wire Line
-	7900 3450 7900 3600
-Wire Wire Line
-	8400 3450 8400 3600
-Wire Wire Line
-	9000 2900 7400 2900
-Wire Wire Line
-	7400 2900 7400 3050
-Wire Wire Line
-	7900 3050 7900 2900
-Connection ~ 7900 2900
-Wire Wire Line
-	8400 3050 8400 2900
-Connection ~ 8400 2900
-Wire Wire Line
-	7100 3150 7100 3250
-Wire Wire Line
-	7600 3150 7600 3250
-Wire Wire Line
-	8100 3150 8100 3250
+	7900 2950 7900 3600
+Wire Wire Line
+	8400 2950 8400 3600
 Wire Wire Line
 	8100 2950 8100 2650
@@
 	7600 2950 7600 2650
 Wire Wire Line
-	7100 2650 7100 2950
+	7100 2650 7100 3450
 Wire Wire Line
 	2300 3200 2500 3200
@@
 Wire Wire Line
 	1400 4850 1550 4850
+Wire Wire Line
+	8100 2950 8400 2950
+Wire Wire Line
+	7600 2950 7900 2950
+Wire Wire Line
+	7100 3450 7400 3450
 $EndSCHEMATC

Commit message: start
Parts:
- AFF1: footprint mylibpcb:indicator_3cif -> myowndevice:indicator_3cif
- J2: footprint mylibpcb:usb5s -> myowndevice:usb5s
Changed lines of the file:
@@
 F 0 "AFF1" H 8100 5100 50  0000 C CNN
 F 1 "CA56-12" H 8100 5000 50  0000 C CNN
-F 2 "mylibpcb:indicator_3cif" H 7600 4300 50  0001 C CNN
+F 2 "myowndevice:indicator_3cif" H 7600 4300 50  0001 C CNN
 F 3 "" H 7600 4300 50  0000 C CNN
 	1    8100 4300
@@
 F 0 "J2" H 2500 5450 50  0000 L CNN
 F 1 "USB_OTG" H 2500 5350 50  0000 L CNN
-F 2 "mylibpcb:usb5s" H 2850 4950 50  0001 C CNN
+F 2 "myowndevice:usb5s" H 2850 4950 50  0001 C CNN
 F 3 "" H 2850 4950 50  0001 C CNN
 	1    2700 5000

Commit message: start
Parts:
- removed J3: CONN_01X02, Pin_Headers:Pin_Header_Angled_1x02_Pitch2.54mm, symbol CONN_01X02
- removed R10, R12, R13, R4, R5, R6, R8, R9: 1k, Resistors_SMD:R_0603_HandSoldering, symbol R_Small
- added J3: Conn_01x01, myowndevice:1pin_sq, symbol timer-rescue:Conn_01x01
- added J4: max809, TO_SOT_Packages_SMD:SOT-23, symbol timer-rescue:Conn_01x03
- added Q1: IRLML6244TRPBF, TO_SOT_Packages_SMD:SOT-23, symbol timer-rescue:Q_NMOS_GSD
- added R1, R3, R4: 200, Resistors_SMD:R_0603_HandSoldering, symbol timer-rescue:R_Small
- added R5: 10k, Resistors_SMD:R_0603_HandSoldering, symbol timer-rescue:R_Small
- added R6: 1k, Resistors_SMD:R_0603_HandSoldering, symbol timer-rescue:R_Small
- added R7: 100k (n.c.), Resistors_SMD:R_0603_HandSoldering, symbol timer-rescue:R_Small
- AFF1: symbol CA56-12 -> timer-rescue:CA56-12
- C1, C2, C3, C4, C5: symbol C_Small -> timer-rescue:C_Small
- D1: symbol LED -> timer-rescue:LED
- IC1: symbol STM8S003F3P -> timer-rescue:STM8S003F3P
- J1: footprint mylibpcb:hc0903a -> myowndevice:hc0903a; symbol CONN_01X02 -> timer-rescue:CONN_01X02
- J2: symbol USB_OTG -> timer-rescue:USB_OTG
- P1, P2: symbol CONN_01X02 -> timer-rescue:CONN_01X02
- P3: footprint Buttons_Switches_THT:SW_Tactile_SKHH_Angled -> Buttons_Switches_ThroughHole:SW_PUSH_6mm_h8mm; symbol CONN_01X02 -> timer-rescue:CONN_01X02
- Q4: symbol Q_NMOS_GSD -> timer-rescue:Q_NMOS_GSD
- R11, R14: symbol R_Small -> timer-rescue:R_Small
- R2: value 10k -> 30k (40ma); symbol R_Small -> timer-rescue:R_Small
- U1: symbol TP4056 -> timer-rescue:TP4056-RESCUE-timer
Connections:
- net GND: now also U1.1 (TEMP), Q1.3 (D), R5.2; no longer P1.2 (P2), P2.2 (P2)
- net VDD: now also J1.2 (P2), P1.1 (P1), P2.2 (P2), J4.3 (Pin_3); no longer J1.1 (P1), P2.1 (P1)
- net a: now also AFF1.11 (a), IC1.12 ([ADC_ETR]I2C_SCL/PB4); no longer IC1.3 (PD6/AIN6/UART1_RX)
- net b: now also AFF1.7 (b), IC1.5 (OSCIN/PA1); no longer IC1.16 ([TIM1_CH1]SPI_MOSI/PC6)
- net c: now also AFF1.4 (c), IC1.16 ([TIM1_CH1]SPI_MOSI/PC6); no longer IC1.13 ([TIM1_CH1N]TIM1_CH3/PC3)
- net c1: now also IC1.13 ([TIM1_CH1N]TIM1_CH3/PC3), R1.1; no longer AFF1.12 (CA1), IC1.2 (PD5/AIN5/UART1_TX)
- net c2: now also IC1.2 (PD5/AIN5/UART1_TX), R3.1; no longer AFF1.9 (CA2), IC1.15 ([TIM2_CH1]SPI_SCK/PC5)
- net c3: now also IC1.3 (PD6/AIN6/UART1_RX), R4.1; no longer AFF1.8 (CA3), IC1.17 ([TIM1_CH2]SPI_MISO/PC7)
- net d: now also AFF1.2 (d), IC1.20 (PD3/AIN4/TIM2_CH2); no longer IC1.12 ([ADC_ETR]I2C_SCL/PB4)
- net dp: now also AFF1.3 (DP), IC1.17 ([TIM1_CH2]SPI_MISO/PC7); no longer IC1.11 ([TIM1_BKIN]I2C_SDA/PB5)
- net e: now also AFF1.1 (e), IC1.19 (PD2/AIN3[TIM2_CH3]); no longer IC1.10 ([SPI_NSS]TIM2_CH3/PA3)
- net f: now also AFF1.10 (f), IC1.14 ([TIM1_CH2N]AIN2/TIM1_CH4/PC4); no longer IC1.5 (OSCIN/PA1)
- net g: now also AFF1.5 (g), IC1.15 ([TIM2_CH1]SPI_SCK/PC5); no longer IC1.14 ([TIM1_CH2N]AIN2/TIM1_CH4/PC4)
- net kn: now also IC1.6 (OSCOUT/PA2); no longer IC1.19 (PD2/AIN3[TIM2_CH3])
- net kn2: now also IC1.11 ([TIM1_BKIN]I2C_SDA/PB5), P1.2 (P2), R5.1; no longer IC1.20 (PD3/AIN4/TIM2_CH2), P1.1 (P1)
- net prg: now also J3.1 (Pin_1)
- net at Q4.3 (D): now also J1.1 (P1); no longer J1.2 (P2)
- new net: AFF1.12 (CA1), R1.2
- new net: AFF1.8 (CA3), R4.2
- new net: AFF1.9 (CA2), R3.2
- new net: J4.1 (Pin_1), P2.1 (P1), Q1.2 (S), R7.1
- new net: Q1.1 (G), R6.1, R7.2
- new net: J4.2 (Pin_2), R6.2
Other:
- moved on the sheet: J1, P2
